Commit message: Fix mesh paths

File: urdf/m710ic70.urdf (robot description, URDF)
Before this commit: robot m710ic70, 10 links, 9 joints
Links:
- link base_link: geometry collision mesh filename=package://fanuc_m710ic_description/meshes/m710ic50/collisio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; visual mesh filename=package://fanuc_m710ic_description/meshes/m710ic50/visual/b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
- link link_1: geometry collision mesh filename=package://fanuc_m710ic_description/meshes/m710ic50/collisio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; visual mesh filename=package://fanuc_m710ic_description/meshes/m710ic50/visual/l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
- link link_2: geometry collision mesh filename=package://fanuc_m710ic_description/meshes/m710ic50/collisio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; visual mesh filename=package://fanuc_m710ic_description/meshes/m710ic50/visual/l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
- link link_3: geometry collision mesh filename=package://fanuc_m710ic_description/meshes/m710ic50/collisio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; visual mesh filename=package://fanuc_m710ic_description/meshes/m710ic50/visual/l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
- link link_4: geometry collision mesh filename=package://fanuc_m710ic_description/meshes/m710ic50/collisio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; visual mesh filename=package://fanuc_m710ic_description/meshes/m710ic50/visual/l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
- link link_5: geometry collision mesh filename=package://fanuc_m710ic_description/meshes/m710ic50/collisio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; visual mesh filename=package://fanuc_m710ic_description/meshes/m710ic50/visual/l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
- link link_6: geometry collision mesh filename=package://fanuc_m710ic_description/meshes/m710ic50/collisio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; visual mesh filename=package://fanuc_m710ic_description/meshes/m710ic50/visual/l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
